File: Hall.kicad_pcb (KiCad board)
At the start: 2 copper layers, 62 x 45.2 mm, 5 parts, among them J1 Conn_01x03_Pin

Commit message: Add files via upload
Routing:
- net GND1: track 0.00 -> 16.0 mm
- added copper zone on B.Cu, net /IP+
- added copper zone on F.Cu, net /IP+
- added copper zone on B.Cu, net GND1
- added copper zone on F.Cu, net GND1
Other:
- outline, holes or cut-outs redrawn
- board text added: "File Format: KICAD 7.0 Material: FR4 Board Thickness: 1mm Copper Foil Thickness: 4 ounces (140um) Green Solder Mask, White Silkscreen, Surface Finish: Electroless Nickel/Immersion Gold Number of Layers: 2 layers"
Changed lines of the file:
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@@
 (kicad_pcb (version 20221018) (generator pcbnew)
   (general
-    (thickness 1.6)
+    (thickness 1)
   )
   (paper "A4")
@@
       (layer "F.Mask" (type "Top Solder Mask") (thickness 0.01))
       (layer "F.Cu" (type "copper") (thickness 0.035))
-      (layer "dielectric 1" (type "core") (thickness 1.51) (material "FR4") (epsilon_r 4.5) (loss_tangent 0.02))
+      (layer "dielectric 1" (type "core") (thickness 0.91) (material "FR4") (epsilon_r 4.5) (loss_tangent 0.02))
       (layer "B.Cu" (type "copper") (thickness 0.035))
       (layer "B.Mask" (type "Bottom Solder Mask") (thickness 0.01))
       (layer "B.Paste" (type "Bottom Solder Paste"))
       (layer "B.SilkS" (type "Bottom Silk Screen"))
-      (copper_finish "None")
+      (copper_finish "Immersion gold")
       (dielectric_constraints no)
     )
     (pad_to_mask_clearance 0)
-    (aux_axis_origin 114.1 86.7)
-    (grid_origin 114.1 86.7)
+    (aux_axis_origin 114.1 0)
+    (grid_origin 114.1 0)
     (pcbplotparams
       (layerselection 0x00010fc_ffffffff)
@@
     (property "ki_keywords" "cap capacitor")
     (attr smd)
-    (fp_text reference "C1" (at -0.06 1.11 90) (layer "F.SilkS")
+    (fp_text reference "C1" (at -0.085 1.5 -180) (layer "F.SilkS")
         (effects (font (size 1 1) (thickness 0.15)))
     )
@@
     (property "ki_keywords" "connector")
     (attr through_hole)
-    (fp_text reference "J1" (at 2.33 4.855) (layer "F.SilkS")
+    (fp_text reference "J1" (at 8.07 0.14) (layer "F.SilkS")
         (effects (font (size 1 1) (thickness 0.15)))
     )
@@
     (property "ki_description" "200kHz, 1.5% Max Tolerance, 100  Internal Resistance Module-alternative Current Sensor for High Current and High Voltage Applications")
     (attr through_hole)
-    (fp_text reference "US1" (at 1.71 -13.84) (layer "F.SilkS")
+    (fp_text reference "US1" (at -5.5 -5.87) (layer "F.SilkS")
         (effects (font (size 1.27 1.27) (thickness 0.254)))
     )
@@
     (property "ki_keywords" "cap capacitor")
     (attr smd)
-    (fp_text reference "C2" (at 0 -1.05) (layer "F.SilkS")
+    (fp_text reference "C2" (at 0.14 -1.14) (layer "F.SilkS")
         (effects (font (size 1 1) (thickness 0.15)))
     )
@@
     (property "ki_keywords" "R res resistor")
     (attr smd)
-    (fp_text reference "R1" (at 0.1 1.28) (layer "F.SilkS")
+    (fp_text reference "R1" (at 0.18 1.07) (layer "F.SilkS")
         (effects (font (size 1 1) (thickness 0.15)))
     )
@@
   (gr_rect (start 114.6 63.02) (end 145.18 80.74)
     (stroke (width 0.15) (type default)) (fill none) (layer "F.SilkS"))
+  (gr_circle (center 140.57 97.09) (end 143.87 97.09)
+    (stroke (width 0.15) (type default)) (fill none) (layer "Edge.Cuts"))
   (gr_rect (start 83.2 63) (end 145.18 108.2)
     (stroke (width 0.15) (type default)) (fill none) (layer "Edge.Cuts"))
+  (gr_circle (center 88.64 96.84) (end 91.94 96.84)
+    (stroke (width 0.15) (type default)) (fill none) (layer "Edge.Cuts"))
+  (gr_text "File Format: KICAD 7.0\nMaterial: FR4\nBoard Thickness: 1mm\nCopper Foil Thickness: 4 ounces (140um)\nGreen Solder Mask, White Silkscreen, \nSurface Finish: Electroless Nickel/Immersion Gold\nNumber of Layers: 2 layers" (at 94.98 123.05) (layer "F.SilkS")
+    (effects (font (size 1 1) (thickness 0.15)) (justify left bottom))
+  )
+  (dimension (type aligned) (layer "F.SilkS")
+    (pts (xy 83.2 108.2) (xy 145.18 108.2))
+    (height 3.26)
+    (gr_text "61.9800 mm" (at 114.19 110.31) (layer "F.SilkS")
+      (effects (font (size 1 1) (thickness 0.15)))
+    )
+    (format (prefix "") (suffix "") (units 3) (units_format 1) (precision 4))
+    (style (thickness 0.15) (arrow_length 1.27) (text_position_mode 0) (extension_height 0.58642) (extension_offset 0.5) keep_text_aligned)
+  )
+  (dimension (type aligned) (layer "F.SilkS")
+    (pts (xy 145.18 63) (xy 145.19 108.19))
+    (height -6.035132)
+    (gr_text "45.1900 mm" (at 152.370132 85.59341 270.0126789) (layer "F.SilkS")
+      (effects (font (size 1 1) (thickness 0.15)))
+    )
+    (format (prefix "") (suffix "") (units 3) (units_format 1) (precision 4))
+    (style (thickness 0.15) (arrow_length 1.27) (text_position_mode 0) (extension_height 0.58642) (extension_offset 0.5) keep_text_aligned)
+  )
   (segment (start 113.405 104.38) (end 127.96 104.38) (width 0.5) (layer "F.Cu") (net 1))
   (segment (start 127.96 104.38) (end 127.99 104.35) (width 0.5) (layer "F.Cu") (net 1))
   (segment (start 112.17 98.535) (end 112.17 103.145) (width 0.5) (layer "F.Cu") (net 1))
   (segment (start 112.17 103.145) (end 113.405 104.38) (width 0.5) (layer "F.Cu") (net 1))
+  (segment (start 130.53 102.34) (end 130.52 102.33) (width 1.2) (layer "F.Cu") (net 2))
+  (segment (start 130.53 106.25) (end 130.53 104.35) (width 1.2) (layer "F.Cu") (net 2))
+  (segment (start 114.1 98.3) (end 114.1 96.66) (width 1.5) (layer "F.Cu") (net 2))
+  (segment (start 130.53 104.35) (end 130.53 102.34) (width 1.2) (layer "F.Cu") (net 2))
+  (segment (start 114.1 98.3) (end 114.1 100.76) (width 1.5) (layer "F.Cu") (net 2))
+  (segment (start 133.7875 100.12) (end 133.7875 99.2125) (width 0.4) (layer "F.Cu") (net 2))
+  (segment (start 130.53 106.25) (end 130.56 106.28) (width 1.2) (layer "F.Cu") (net 2))
+  (segment (start 130.53 104.35) (end 130.53 105.99) (width 1.5) (layer "B.Cu") (net 2))
+  (segment (start 130.53 104.35) (end 130.53 102.48) (width 1.5) (layer "B.Cu") (net 2))
+  (segment (start 114.1 98.3) (end 114.1 96.46) (width 1.5) (layer "B.Cu") (net 2))
+  (segment (start 114.1 98.3) (end 114.1 100) (width 1.5) (layer "B.Cu") (net 2))
   (segment (start 132.9725 100.12) (end 132.07 100.12) (width 0.4) (layer "F.Cu") (net 3))
   (segment (start 133.07 100.14) (end 133.07 104.35) (width 0.4) (layer "F.Cu") (net 3))
   (segment (start 131.37 100.13) (end 129.54 98.3) (width 0.5) (layer "F.Cu") (net 4))
   (segment (start 129.54 98.3) (end 116.01 98.3) (width 0.5) (layer "F.Cu") (net 4))
+  (zone (net 5) (net_name "/IP+") (layers "F&B.Cu") (hatch edge 0.5)
+    (priority 1)
+    (connect_pads (clearance 0.5))
+    (min_thickness 0.25) (filled_areas_thickness no)
+    (fill yes (thermal_gap 0.5) (thermal_bridge_width 0.5))
+    (polygon
+      (pts
+        (xy 114.62 62.98)
+        (xy 145.18 62.97)
+        (xy 145.16 80.74)
+        (xy 114.6 80.69)
+      )
+    )
+  )
   (zone (net 6) (net_name "/IP-") (layers "F&B.Cu") (hatch edge 0.5)
     (connect_pads (clearance 0))
     (min_thickness 0.25) (filled_areas_thickness no)
-    (fill (thermal_gap 0.5) (thermal_bridge_width 0.5))
+    (fill yes (thermal_gap 0.5) (thermal_bridge_width 0.5))
     (polygon
       (pts
@@
       )
     )
+  )
+  (zone (net 2) (net_name "GND1") (layers "F&B.Cu") (hatch edge 0.5)
+    (priority 2)
+    (connect_pads (clearance 0.5))
+    (min_thickness 0.25) (filled_areas_thickness no)
+    (fill yes (thermal_gap 0.5) (thermal_bridge_width 0.5))
+    (polygon
+      (pts
+        (xy 83.24 80.78)
+        (xy 83.19 108.18)
+        (xy 145.19 108.19)
+        (xy 145.16 80.74)
+      )
+    )
+  )
+  (zone (net 0) (net_name "") (layers "*.Paste") (hatch full 0.5)
+    (connect_pads (clearance 0.5))
+    (min_thickness 0.25) (filled_areas_thickness no)
+    (fill yes (thermal_gap 0.5) (thermal_bridge_width 0.5))
+    (polygon
+      (pts
+        (xy 113.85 80.25)
+        (xy 113.77 62.97)
+        (xy 83.15 63.02)
+        (xy 83.22 80.25)
+      )
+    )
+  )
+  (zone (net 0) (net_name "") (layers "*.Paste") (hatch full 0.5)
+    (connect_pads (clearance 0.5))
+    (min_thickness 0.25) (filled_areas_thickness no)
+    (fill yes (thermal_gap 0.5) (thermal_bridge_width 0.5))
+    (polygon
+      (pts
+        (xy 114.59 63)
+        (xy 114.59 80.2)
+        (xy 145.16 80.23)
+        (xy 145.18 62.97)
+      )
+    )

Commit message: Add files via upload
Parts:
- C1: footprint Capacitor_SMD:C_0201_0603Metric -> Capacitor_SMD:C_0603_1608Metric
- C2: footprint Capacitor_SMD:C_0201_0603Metric_Pad0.64x0.40mm_HandSolder -> Capacitor_SMD:C_0603_1608Metric
- R1: footprint Resistor_SMD:R_0201_0603Metric -> Resistor_SMD:R_0603_1608Metric
- moved J1 16.4 mm to (111.6, 104.6)
- moved C1 16.1 mm to (108.5, 105.4), turned to 90 degrees
- moved C2 13.1 mm to (121.2, 104.8)
- moved R1 11.5 mm to (120.4, 102.4), turned to 90 degrees
Routing:
- net Net-(US1-VIOUT): track 16.1 -> 5.77 mm
- net VCC: track 21.0 -> 10.8 mm
- net GND1: track 16.0 -> 14.6 mm
