File: Veronte68BreakOut.kicad_pcb (KiCad board)
At the start: 2 copper layers, 125 x 200 mm, 12 parts, among them J1 DC37_Receptacle_MountingHoles, J10 Barrel_Jack_Switch, J11 Barrel_Jack_Switch, J2 DC37_Receptacle_MountingHoles, J3 DE9_Receptacle_MountingHoles, J4 Conn_01x19, J5 Conn_01x11, J6 Conn_01x19, J7 Conn_01x13, J8 Conn_01x06

Commit message: add v2.0
add v2.0
Connections:
- J2 pad 22: GND -> Net-(J7-Pin_3)
- J7 pad 3: GND -> Net-(J7-Pin_3)
Routing:
- net Net-(J7-Pin_3): track 0.00 -> 113.8 mm
- net GND: track 1143.5 -> 1029.7 mm
Other:
- board text added: "Veronte 68 pin to 2.54mm pitch adapter BRD v2.0 20230801 teTra aviation corp."
- board text removed: "Veronte 68 pin to 2.54mm pitch adapter BRD v1.3.0 20230707 teTra aviation corp."
Changed lines of the file:
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@@
   (paper "A3" portrait)
   (title_block
-    (date "2023-07-07")
-    (rev "V1.1")
+    (title "Veronte68BreakOut")
+    (date "2023-08-01")
+    (rev "V2.0")
     (company "teTra Aviation Corp.")
   )
@@
   (net 73 "unconnected-(J3-Pad8)")
   (net 74 "GND")
+  (net 75 "Net-(J7-Pin_3)")
   (footprint "LOGO" (layer "F.Cu")
     (at 102.87 86.995)
@@
       (net 50 "Net-(J7-Pin_2)") (pinfunction "21") (pintype "passive"))
     (pad "22" thru_hole circle (at -6.925 2.84 90) (size 1.6 1.6) (drill 1) (layers "*.Cu" "*.Mask")
-      (net 74 "GND") (pinfunction "22") (pintype "passive"))
+      (net 75 "Net-(J7-Pin_3)") (pinfunction "22") (pintype "passive"))
     (pad "23" thru_hole circle (at -9.695 2.84 90) (size 1.6 1.6) (drill 1) (layers "*.Cu" "*.Mask")
       (net 51 "Net-(J7-Pin_4)") (pinfunction "23") (pintype "passive"))
@@
       (net 50 "Net-(J7-Pin_2)") (pinfunction "Pin_2") (pintype "passive"))
     (pad "3" thru_hole oval (at 0 5.08) (size 1.7 1.7) (drill 1) (layers "*.Cu" "*.Mask")
-      (net 74 "GND") (pinfunction "Pin_3") (pintype "passive"))
+      (net 75 "Net-(J7-Pin_3)") (pinfunction "Pin_3") (pintype "passive"))
     (pad "4" thru_hole oval (at 0 7.62) (size 1.7 1.7) (drill 1) (layers "*.Cu" "*.Mask")
       (net 51 "Net-(J7-Pin_4)") (pinfunction "Pin_4") (pintype "passive"))
@@
     (effects (font (size 1.58 1.58) (thickness 0.15)) (justify left bottom))
   )
-  (gr_text "Veronte 68 pin to 2.54mm pitch adapter BRD\nv1.3.0 20230707\nteTra aviation corp." (at 104.14 108.585) (layer "F.SilkS")
+  (gr_text "Veronte 68 pin to 2.54mm pitch adapter BRD\nv2.0 20230801\nteTra aviation corp." (at 104.14 108.585) (layer "F.SilkS")
     (effects (font (size 1.58 1.58) (thickness 0.15)))
   )
@@
   (segment (start 101.13 198.17) (end 186.63 198.17) (width 2) (layer "F.Cu") (net 69))
   (segment (start 73.66 55.88) (end 74.8369 55.88) (width 0.25) (layer "F.Cu") (net 74))
-  (segment (start 76.0506 130.7537) (end 74.8369 129.54) (width 0.25) (layer "F.Cu") (net 74))
   (segment (start 128.435 41.455) (end 186.84 41.455) (width 0.25) (layer "F.Cu") (net 74))
   (segment (start 127 134.62) (end 128.1769 134.62) (width 0.25) (layer "F.Cu") (net 74))
-  (segment (start 186.6713 130.7537) (end 76.0506 130.7537) (width 0.25) (layer "F.Cu") (net 74))
   (segment (start 74.8369 55.88) (end 76.0138 57.0569) (width 0.25) (layer "F.Cu") (net 74))
   (segment (start 180.89 81.28) (end 184 84.39) (width 0.25) (layer "F.Cu") (net 74))
-  (segment (start 73.66 129.54) (end 74.8369 129.54) (width 0.25) (layer "F.Cu") (net 74))
   (segment (start 76.0138 57.0569) (end 154.9756 57.0569) (width 0.25) (layer "F.Cu") (net 74))
   (segment (start 184 134.74) (end 128.2969 134.74) (width 0.25) (layer "F.Cu") (net 74))
@@
   (segment (start 184 140.28) (end 133.0156 140.28) (width 0.25) (layer "F.Cu") (net 74))
   (segment (start 128.0369 41.8531) (end 128.435 41.455) (width 0.25) (layer "F.Cu") (net 74))
-  (segment (start 186.84 130.585) (end 186.6713 130.7537) (width 0.25) (layer "F.Cu") (net 74))
   (segment (start 184 151.36) (end 183.2265 150.5865) (width 0.25) (layer "F.Cu") (net 74))
   (segment (start 182.7752 158.4452) (end 127.9652 158.4452) (width 0.25) (layer "F.Cu") (net 74))
@@
   (segment (start 76.0153 64.6784) (end 157.6604 64.6784) (width 0.25) (layer "F.Cu") (net 74))
   (segment (start 162.3019 148.4969) (end 163.78 149.975) (width 0.25) (layer "F.Cu") (net 74))
+  (segment (start 76.0506 130.7537) (end 74.8369 129.54) (width 0.25) (layer "F.Cu") (net 75))
+  (segment (start 186.6713 130.7537) (end 76.0506 130.7537) (width 0.25) (layer "F.Cu") (net 75))
+  (segment (start 73.66 129.54) (end 74.8369 129.54) (width 0.25) (layer "F.Cu") (net 75))
+  (segment (start 186.84 130.585) (end 186.6713 130.7537) (width 0.25) (layer "F.Cu") (net 75))
   (zone (net 74) (net_name "GND") (layers "F&B.Cu") (hatch edge 0.5)
     (connect_pads (clearance 0.5))
